File: GHDR_Main.kicad_sch (KiCad schematic)
At the start: 77 parts, among them J300 EXT UART Connector, J301 STM32 Debug Connection, J302 Buzzer Connector, J303 EXT SPI Connector, J304 EXT I2C Connector, J305 (M) Power & ESC Connector, J306 (M) AUX Connector Main Board, J307 EXT GPS Connector, J308 EXT 5V, J309 EXT USART1, Q300 MMBT3904, SW300 TACTILE SWITCH, SW301 TACTILE SWITCH, U300 SP1117, U301 W25Q128JVPIQTR, U302 BMP580, U303 ICM-42670-P, U304 STM32H743VITx, X300 XVFEELNANF-8MHZ

Commit message: feat: update
Parts:
- added C202: 2.2uF, Capacitor_SMD:C_0805_2012Metric, symbol Device:C_Small
- added C208: 100uF, Capacitor_SMD:C_1206_3216Metric, symbol Device:C_Small
- added Q200: AO3011A, easyeda2kicad:SOT-23-3_L2.9-W1.6-P1.90-LS2.8-BR, symbol easyeda2kicad:AO3011A
- added TP200, TP202: TestPoint, TestPoint:TestPoint_Pad_D1.5mm, symbol Connector:TestPoint
- added TP201: TestPoint, TestPoint:TestPoint_Pad_D1.0mm, symbol Connector:TestPoint
- added U200: MX74610T, easyeda2kicad:SOT-23-6_L2.9-W1.6-P0.95-LS2.8-BL-1, symbol easyeda2kicad:MX74610T
- renumbered C306 to C200, C302 to C201, C300 to C203, C303 to C204, C301 to C205, C309 to C206, C305 to C207, C307 to C209, C304 to C210, C311 to C211, C310 to C212, C308 to C213, C312 to C214, C316 to C215, C314 to C216, C313 to C217, C315 to C218, C318 to C219, C319 to C220, C317 to C221, C320 to C222, C323 to C223, C322 to C224, C324 to C225, C325 to C226, C321 to C227, C327 to C228, C328 to C229, C330 to C230, C329 to C231, C326 to C232, C331 to C233, Card300 to Card200, D300 to D200, D301 to D201, FB300 to FB200, FB301 to FB201, J301 to J200, J300 to J201, J302 to J202, J303 to J203, J305 to J204, J306 to J205, J308 to J206, J304 to J207, J309 to J208, J307 to J209, LED300 to LED200, LED301 to LED201, Q300 to Q201, R300 to R200, R304 to R201, R303 to R202, R302 to R203, R305 to R204, R306 to R205, R308 to R206, R307 to R207, R310 to R208, R309 to R209, R312 to R210, R311 to R211, R301 to R212, R315 to R213, R316 to R214, R313 to R215, R314 to R216, R317 to R217, SW300 to SW200, SW301 to SW201, U300 to U201, U301 to U202, U302 to U203, U303 to U204, U304 to U205, USB300 to USB200, X300 to X200
Connections:
- net +3.3V: now also TP202.1
- net +5V: now also C208.1, Q200.3 (D), TP200.1, U200.1 (CATHODE); no longer D200.1 (K), J201.1 (Pin_1), J202.1 (Pin_1), J203.1 (Pin_1), J204.1 (Pin_1), J206.1 (Pin_1), J207.1 (Pin_1), J209.1 (Pin_1)
- net +USB_VBUS: now also TP201.1
- net GND: now also J201.1 (Pin_1), J203.1 (Pin_1), J204.1 (Pin_1), J206.1 (Pin_1), J207.1 (Pin_1), J209.1 (Pin_1), C208.2; no longer J201.2 (Pin_2), J203.2 (Pin_2), J204.2 (Pin_2), J206.2 (Pin_2), J207.2 (Pin_2), J209.2 (Pin_2)
- net at D201.1 (K): now also J202.1 (Pin_1); no longer J202.2 (Pin_2)
- new net: C202.1, U200.6 (VCAPL)
- new net: C202.2, U200.5 (VCAPH)
- new net: Q200.1 (G), U200.2 (GATEPD), U200.3 (GATE)
- new net +5V_RAW: D200.1 (K), J201.2 (Pin_2), J202.2 (Pin_2), J203.2 (Pin_2), J204.2 (Pin_2), J206.2 (Pin_2), J207.2 (Pin_2), J209.2 (Pin_2), Q200.2 (S), U200.4 (ANODE)
Other:
- note added: "+5V Protection"
- note added: "Test Points"
- moved on the sheet: C200, C203, C205, D200, D201, J202, J206, Q201, R204

Commit message: feat: update for github
Parts:
- removed C200, C203, C205, C208: 100uF, Capacitor_SMD:C_1206_3216Metric, symbol Device:C_Small
- removed LED200: XL-1608PGC-06, easyeda2kicad:LED0603-RD_GREEN, symbol easyeda2kicad:XL-1608PGC-06
- removed LED201: NCD0603R1, easyeda2kicad:LED0603-RD_RED, symbol easyeda2kicad:FC-DA1608HRK-620D
- added C210: 10TPE220ML, easyeda2kicad:CAP-SMD_L7.3-W4.3, symbol easyeda2kicad:10TPE220ML
- added D200, D203: LED, LED_SMD:LED_0603_1608Metric, symbol Device:LED
- D201: renamed from D200; Manfufacture ID (none) -> DSK34
- J200: renamed from J201; now left out of the parts list
- J202: renamed from J203; now left out of the parts list
- J203: renamed from J202; now left out of the parts list
- J204, J208, J209, TP200, TP201, TP202: now left out of the parts list
- J205: renamed from J207; now left out of the parts list
- J206: renamed from J205; now left out of the parts list
- J207: renamed from J206; now left out of the parts list
- R202: renamed from R203; LCSC Part C25804 -> C269716
- R204: renamed from R200; LCSC Part C25804 -> C269716
- R212: LCSC Part C125768 -> C22962; Manfufacture ID RS-03K3300FT -> 0603WAF2200T5E
- U203: Manfufacture ID (none) -> W25Q128JVPIQTR
- U205: renamed from U204; Manfufacture ID (none) -> ICM-42670-P
- renumbered C201 to C200, C211 to C201, C206 to C203, C209 to C204, C213 to C205, C210 to C206, C204 to C208, C212 to C209, C214 to C211, C217 to C212, C218 to C213, C216 to C214, C221 to C215, C219 to C216, C220 to C217, C215 to C218, C224 to C219, C222 to C220, C223 to C221, C232 to C222, C225 to C223, C226 to C224, C229 to C225, C228 to C226, C230 to C227, C231 to C228, C227 to C229, C233 to C230, D201 to D202, J200 to J201, R201 to R200, R202 to R201, R204 to R203, R217 to R214, R214 to R215, R215 to R217, U205 to U204
Connections:
- net +5V: now also C210.1
- net GND: now also C210.2, D200.1 (K), D203.1 (K)
- net at R212.2: now also D203.2 (A)
- net at R207.2: now also D200.2 (A)
