File: GHDR_Main.kicad_sch (KiCad schematic)
At the start: 81 parts, among them J200 EXT UART Connector, J201 STM32 Debug Connection, J202 EXT SPI Connector, J203 Buzzer Connector, J204 (M) Power & ESC Connector, J205 EXT I2C Connector, J206 (M) AUX Connector Main Board, J207 EXT 5V, J208 EXT USART1, J209 EXT GPS Connector, Q200 AO3011A, Q201 MMBT3904, SW200 TACTILE SWITCH, SW201 TACTILE SWITCH, U200 MX74610T, U201 SP1117, U202 W25Q128JVPIQTR, U203 BMP580, U204 STM32H743VITx, U205 ICM-42670-P, X200 XVFEELNANF-8MHZ

Commit message: feat: change crystal
Parts:
- removed X200: XVFEELNANF-8MHZ, easyeda2kicad:CRYSTAL-SMD_4P-L5.0-W3.2-BL-1, symbol easyeda2kicad:XVFEELNANF-8MHZ
- added X201: X32258MOB4SI, easyeda2kicad:CRYSTAL-SMD_4P-L3.2-W2.5-BL, symbol easyeda2kicad:X32258MOB4SI
- C200, C218: value 22pF -> 18pF
- R206: value 10K -> 1K
Connections:
- net +3.3V: no longer R212.1
- net GND: now also X201.2 (GND), X201.4 (GND)
- net STM32_NRST: now also R212.1
- net STM32_XTAL_IN: now also X201.1
- net STM32_XTAL_OUT: now also X201.3
Other:
- moved on the sheet: D203, R212
Changed lines of the file:
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@@
 	(wire
 		(pts
-			(xy 384.81 127) (xy 388.62 127)
+			(xy 389.89 127) (xy 393.7 127)
 		)
 		(stroke
@@
 	(wire
 		(pts
-			(xy 373.38 127) (xy 377.19 127)
+			(xy 378.46 127) (xy 382.27 127)
 		)
 		(stroke
@@
 	(global_label "GND"
 		(shape input)
-		(at 388.62 127 0)
+		(at 393.7 127 0)
 		(fields_autoplaced yes)
 		(effects
@@
 		)
 		(property "Intersheetrefs" "${INTERSHEET_REFS}"
-			(at 394.0179 127 0)
+			(at 399.0979 127 0)
 			(effects
 				(font
@@
 		)
 	)
-	(global_label "+3.3V"
-		(shape input)
-		(at 368.3 127 180)
-		(fields_autoplaced yes)
-		(effects
-			(font
-				(size 1 1)
-			)
-			(justify right)
-		)
-		(property "Intersheetrefs" "${INTERSHEET_REFS}"
-			(at 361.4735 127 0)
-			(effects
-				(font
-					(size 1.27 1.27)
-				)
-				(justify right)
-				(hide yes)
-			)
-		)
-	)
 	(global_label "STM32_USART3_TX"
 		(shape bidirectional)
@@
 		)
 	)
+	(global_label "STM32_NRST"
+		(shape input)
+		(at 373.38 127 180)
+		(fields_autoplaced yes)
+		(effects
+			(font
+				(size 1 1)
+			)
+			(justify right)
+		)
+		(property "Intersheetrefs" "${INTERSHEET_REFS}"
+			(at 361.7439 127 0)
+			(effects
+				(font
+					(size 1.27 1.27)
+				)
+				(justify right)
+				(hide yes)
+			)
+		)
+	)
 	(global_label "GND"
 		(shape input)
@@
 	)
 	(symbol
-		(lib_id "easyeda2kicad:XVFEELNANF-8MHZ")
-		(at 46.99 33.02 0)
-		(unit 1)
-		(exclude_from_sim no)
-		(in_bom yes)
-		(on_board yes)
-		(dnp no)
-		(fields_autoplaced yes)
-		(property "Reference" "X200"
-			(at 46.99 22.86 0)
-			(effects
-				(font
-					(size 1 1)
-				)
-			)
-		)
-		(property "Value" "XVFEELNANF-8MHZ"
-			(at 46.99 25.4 0)
-			(effects
-				(font
-					(size 1 1)
-				)
-			)
-		)
-		(property "Footprint" "easyeda2kicad:CRYSTAL-SMD_4P-L5.0-W3.2-BL-1"
-			(at 46.99 43.18 0)
-			(effects
-				(font
-					(size 1.27 1.27)
-				)
-				(hide yes)
-			)
-		)
-		(property "Datasheet" ""
-			(at 46.99 33.02 0)
-			(effects
-				(font
-					(size 1.27 1.27)
-				)
-				(hide yes)
-			)
-		)
-		(property "Description" ""
-			(at 46.99 33.02 0)
-			(effects
-				(font
-					(size 1.27 1.27)
-				)
-				(hide yes)
-			)
-		)
-		(property "LCSC Part" "C5160132"
-			(at 46.99 45.72 0)
-			(effects
-				(font
-					(size 1.27 1.27)
-				)
-				(hide yes)
-			)
-		)
-		(property "Manfufacture ID" "XVFEELNANF-8MHZ"
-			(at 46.99 33.02 0)
-			(effects
-				(font
-					(size 1.27 1.27)
-				)
-				(hide yes)
-			)
-		)
-		(pin "4"
-		)
-		(pin "1"
-		)
-		(pin "3"
-		)
-		(pin "2"
-		)
-		(instances
-			(project "GHDR"
-				(path "/2509eac7-702d-471d-ac76-1a26bd9d0364/2199fe3b-d1e6-4213-a727-a65ad5091fa9"
-					(reference "X?")
-					(unit 1)
-				)
-			)
-			(project "GHDR_Main"
-				(path "/6d288c5b-71e1-494f-b1b1-4e9da334c008"
-					(reference "X200")
-					(unit 1)
-				)
-			)
-		)
-	)
-	(symbol
 		(lib_id "Device:C_Small")
 		(at 223.52 40.64 0)
@@
 			)
 		)
-		(property "Value" "10K"
+		(property "Value" "1K"
 			(at 103.378 39.878 0)
 			(effects
@@
 	(symbol
 		(lib_id "Device:R_Small")
-		(at 370.84 127 90)
+		(at 375.92 127 90)
 		(mirror x)
 		(unit 1)
@@
 		(dnp no)
 		(property "Reference" "R212"
-			(at 370.84 121.92 90)
+			(at 375.92 121.92 90)
 			(effects
 				(font
@@
 		)
 		(property "Value" "220"
-			(at 370.84 124.206 90)
+			(at 375.92 124.206 90)
 			(effects
 				(font
@@
 		)
 		(property "Footprint" "Resistor_SMD:R_0603_1608Metric"
-			(at 370.84 127 0)
+			(at 375.92 127 0)
 			(effects
 				(font
@@
 		)
 		(property "Datasheet" "~"
-			(at 370.84 127 0)
+			(at 375.92 127 0)
 			(effects
 				(font
@@
 		)
 		(property "Description" "Resistor, small symbol"
-			(at 370.84 127 0)
+			(at 375.92 127 0)
 			(effects
 				(font
@@
 		)
 		(property "Manfufacture ID" "0603WAF2200T5E"
-			(at 370.84 127 90)
+			(at 375.92 127 90)
 			(effects
 				(font
@@
 		)
 		(property "LCSC Part" "C22962"
-			(at 370.84 127 90)
+			(at 375.92 127 90)
 			(effects
 				(font
@@
 			)
 		)
-		(property "Value" "22pF"
+		(property "Value" "18pF"
 			(at 32.766 39.37 0)
 			(effects
@@
 	)
 	(symbol
+		(lib_id "easyeda2kicad:X32258MOB4SI")
+		(at 46.99 33.02 0)
+		(unit 1)
+		(exclude_from_sim no)
+		(in_bom yes)
+		(on_board yes)
+		(dnp no)
+		(fields_autoplaced yes)
+		(property "Reference" "X201"
+			(at 46.99 22.86 0)
+			(effects
+				(font
+					(size 1.27 1.27)
+				)
+			)
+		)
+		(property "Value" "X32258MOB4SI"
+			(at 46.99 25.4 0)
+			(effects
+				(font
+					(size 1.27 1.27)
+				)
+			)
+		)
+		(property "Footprint" "easyeda2kicad:CRYSTAL-SMD_4P-L3.2-W2.5-BL"
+			(at 46.99 43.18 0)
+			(effects
+				(font
+					(size 1.27 1.27)
+				)
+				(hide yes)
+			)
+		)
+		(property "Datasheet" ""
+			(at 46.99 33.02 0)
+			(effects
+				(font
+					(size 1.27 1.27)
+				)
+				(hide yes)
+			)
+		)
+		(property "Description" ""
+			(at 46.99 33.02 0)
+			(effects
+				(font
+					(size 1.27 1.27)
+				)
+				(hide yes)
+			)
+		)
+		(property "LCSC Part" "C2682775"
+			(at 46.99 45.72 0)
+			(effects
+				(font
+					(size 1.27 1.27)
+				)
+				(hide yes)
+			)
+		)
+		(pin "2"
+		)
+		(pin "3"
+		)
+		(pin "1"
+		)
+		(pin "4"
+		)
+		(instances
+			(project ""
+				(path "/6d288c5b-71e1-494f-b1b1-4e9da334c008"
+					(reference "X201")
+					(unit 1)
+				)
+			)
+		)
+	)
+	(symbol
 		(lib_id "Device:C_Small")
 		(at 173.99 180.34 0)
@@
 			)
 		)
-		(property "Value" "22pF"
+		(property "Value" "18pF"
 			(at 63.754 28.448 0)
 			(effects
@@
 	(symbol
 		(lib_id "Device:LED")
-		(at 381 127 180)
+		(at 386.08 127 180)
 		(unit 1)
 		(exclude_from_sim no)
@@
 		(dnp no)
 		(property "Reference" "D203"
-			(at 381 120.904 0)
+			(at 386.08 120.904 0)
 			(effects
 				(font
@@
 		)
 		(property "Value" "LED"
-			(at 381 123.444 0)
+			(at 386.08 123.444 0)
 			(effects
 				(font
@@
 		)
 		(property "Footprint" "LED_SMD:LED_0603_1608Metric"
-			(at 381 127 0)
+			(at 386.08 127 0)
 			(effects
 				(font
@@
 		)
 		(property "Datasheet" "~"
-			(at 381 127 0)
+			(at 386.08 127 0)
 			(effects
 				(font
@@
 		)
 		(property "Description" "Light emitting diode"
-			(at 381 127 0)
+			(at 386.08 127 0)
 			(effects
 				(font
@@
 		)
 		(property "Sim.Pins" "1=K 2=A"
-			(at 381 127 0)
+			(at 386.08 127 0)
 			(effects
 				(font
@@
 		)
 		(property "LCSC Part" "C84263"
-			(at 381 127 0)
+			(at 386.08 127 0)
 			(effects
 				(font
@@
 		)
 		(property "Manfufacture ID" "NCD0603R1"
-			(at 381 127 0)
+			(at 386.08 127 0)
 			(effects
 				(font
