File: GHDR_Main.kicad_pcb (KiCad board)
At the start: 4 copper layers, 50 x 70 mm, 84 parts, among them J300 EXT UART Connector, J301 STM32 Debug Connection, J302 Buzzer Connector, J303 EXT SPI Connector, J304 EXT I2C Connector, J305 (M) Power & ESC Connector, J306 (M) AUX Connector Main Board, J307 EXT GPS Connector, J308 EXT 5V, J309 EXT USART1, Q300 MMBT3904, SW300 TACTILE SWITCH, SW301 TACTILE SWITCH, U300 SP1117, U301 W25Q128JVPIQTR, U302 BMP580, U303 ICM-42670-P, U304 STM32H743VITx, X300 XVFEELNANF-8MHZ

Commit message: feat: update
Parts:
- removed C300, C301, C306: 100uF, Capacitor_SMD:C_1206_3216Metric
- removed C303, C311: 10uF, Capacitor_SMD:C_0805_2012Metric
- removed D300: DSK34, easyeda2kicad:SOD-123FL_L2.7-W1.8-LS3.8-RD
- removed LED301: NCD0603R1, easyeda2kicad:LED0603-RD_RED
- removed R301: 220, Resistor_SMD:R_0603_1608Metric
- removed U300: SP1117, Package_TO_SOT_SMD:SOT-223-3_TabPin2
- added C200: 100uF, Capacitor_SMD:C_1206_3216Metric, F.Cu at (137.6, 74.6)
- added C202: 2.2uF, Capacitor_SMD:C_0805_2012Metric, F.Cu at (135.0, 78.5)
- added C203: 100uF, Capacitor_SMD:C_1206_3216Metric, F.Cu at (143.9, 75.0)
- added C204: 10uF, Capacitor_SMD:C_0805_2012Metric, F.Cu at (155.2, 76.5)
- added C205: 100uF, Capacitor_SMD:C_1206_3216Metric, F.Cu at (141.6, 79.7)
- added C208: 100uF, Capacitor_SMD:C_1206_3216Metric, F.Cu at (141.5, 75.0)
- added C211: 10uF, Capacitor_SMD:C_0805_2012Metric, F.Cu at (143.8, 80.3)
- added D200: DSK34, easyeda2kicad:SOD-123FL_L2.7-W1.8-LS3.8-RD, F.Cu at (135.8, 72.0)
- added LED201: NCD0603R1, easyeda2kicad:LED0603-RD_RED, F.Cu at (138.8, 124.2)
- added Q200: AO3011A, easyeda2kicad:SOT-23-3_L2.9-W1.6-P1.90-LS2.8-BR, F.Cu at (135.4, 82.3)
- added R212: 220, Resistor_SMD:R_0603_1608Metric, F.Cu at (137.2, 124.2)
- added TP200: TestPoint, TestPoint:TestPoint_Pad_D1.5mm, F.Cu at (138.9, 82.5)
- added TP201: TestPoint, TestPoint:TestPoint_Pad_D1.0mm, F.Cu at (144.9, 68.5)
- added TP202: TestPoint, TestPoint:TestPoint_Pad_D1.5mm, F.Cu at (160.0, 109.1)
- added U200: MX74610T, easyeda2kicad:SOT-23-6_L2.9-W1.6-P0.95-LS2.8-BL-1, F.Cu at (138.2, 78.5)
- added U201: SP1117, Package_TO_SOT_SMD:SOT-223-3_TabPin2, F.Cu at (149.7, 77.4)
- REF** (x4): value MountingHole_3.5mm_Pad_Via_Custom -> MountingHole_3.5mm_5mm_Pad_Via; footprint easyeda2kicad:MountingHole_3.5mm_Pad_Via_Custom -> easyeda2kicad:MountingHole_3.5mm_5mm_Pad_Via
- moved J203 12.7 mm to (172.3, 85.9), turned to 180 degrees
- moved J209 12.7 mm to (172.3, 123.3), turned to 180 degrees
- moved R201 1.28 mm to (148.9, 82.6)
- moved R202 1.28 mm to (147.3, 82.6)
- renumbered C302 to C201, C309 to C206, C305 to C207, C307 to C209, C304 to C210, C310 to C212, C308 to C213, C312 to C214, C316 to C215, C314 to C216, C313 to C217, C315 to C218, C318 to C219, C319 to C220, C317 to C221, C320 to C222, C323 to C223, C322 to C224, C324 to C225, C325 to C226, C321 to C227, C327 to C228, C328 to C229, C330 to C230, C329 to C231, C326 to C232, C331 to C233, Card300 to Card200, D301 to D201, FB300 to FB200, FB301 to FB201, J301 to J200, J300 to J201, J302 to J202, J303 to J203, J305 to J204, J306 to J205, J308 to J206, J304 to J207, J309 to J208, J307 to J209, LED300 to LED200, Q300 to Q201, R300 to R200, R304 to R201, R303 to R202, R302 to R203, R305 to R204, R306 to R205, R308 to R206, R307 to R207, R310 to R208, R309 to R209, R312 to R210, R311 to R211, R315 to R213, R316 to R214, R313 to R215, R314 to R216, R317 to R217, SW300 to SW200, SW301 to SW201, U301 to U202, U302 to U203, U303 to U204, U304 to U205, USB300 to USB200, X300 to X200
Connections:
- D201 pad 1: Net-(D1-K) -> Net-(D301-K)
- J201 pad 1: +5V -> GND
- J201 pad 2: GND -> +5V_RAW
- J202 pad 1: +5V -> Net-(D301-K)
- J202 pad 2: Net-(D1-K) -> +5V_RAW
- J203 pad 1: +5V -> GND
- J203 pad 2: GND -> +5V_RAW
- J204 pad 1: +5V -> GND
- J204 pad 2: GND -> +5V_RAW
- J206 pad 1: +5V -> GND
- J206 pad 2: GND -> +5V_RAW
- J207 pad 1: +5V -> GND
- J207 pad 2: GND -> +5V_RAW
- J209 pad 1: +5V -> GND
- J209 pad 2: GND -> +5V_RAW
Routing:
- net STM32_ISP2_MOSI: track 19.1 -> 37.9 mm
- net +5V_RAW: track 0.00 -> 17.3 mm, vias 0 -> 1
- net STM32_I2C1_SDA: track 135.2 -> 119.2 mm, vias 2 -> 4
- net STM32_I2C1_SCL: track 128.7 -> 118.6 mm, vias 4 -> 2
- net +USB_VBUS: track 0.00 -> 10.1 mm, vias 0 -> 3
- net STM32_ISP2_MISO: track 24.3 -> 34.2 mm, vias 0 -> 2
- net Net-(D301-K): track 0.00 -> 7.90 mm
- net STM32_USART2_TX: track 53.2 -> 59.3 mm, vias 2 -> 4
- net GND: track 87.1 -> 81.1 mm, vias 33 -> 37
- net Net-(Q1-G): track 0.00 -> 5.72 mm
- net +5V: track 20.0 -> 25.6 mm, vias 1 -> 0
- net Net-(D1-K): track 5.36 -> 0.00 mm
- net +3.3V: track 88.6 -> 85.4 mm, vias 21 -> 24
- net STM32_ISP2_SCK: track 27.7 -> 30.8 mm, vias 0 -> 2
- net STM32_ISP2_NSS: track 30.9 -> 27.9 mm, vias 0 -> 2
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- added copper zone on In2.Cu, net +5V_RAW
- added copper zone on In2.Cu, net +USB_VBUS
- removed copper zone on B.Cu, net +5V
- removed copper zone on F.Cu, net +USB_VBUS
Other:
- board text added: "3V3"
- board text added: "USBV"

Commit message: feat: update for github
Parts:
- removed the C200 at (137.6, 74.6)
- removed the C205 at (141.6, 79.7)
- removed the C208 at (141.5, 75.0)
- removed LED200: XL-1608PGC-06, easyeda2kicad:LED0603-RD_GREEN
- removed LED201: NCD0603R1, easyeda2kicad:LED0603-RD_RED
- added D200: LED, LED_SMD:LED_0603_1608Metric, F.Cu at (139.3, 86.2)
- added D203: LED, LED_SMD:LED_0603_1608Metric, F.Cu at (138.8, 124.2)
- C210: renamed from C203; value 100uF -> 10TPE220ML; footprint Capacitor_SMD:C_1206_3216Metric -> easyeda2kicad:CAP-SMD_L7.3-W4.3
- moved G*** 12.7 mm to (135.6, 97.7)
- moved C201 7.11 mm to (138.5, 75.6), turned to 180 degrees
- moved C210 2.25 mm to (143.2, 77.1), turned to -90 degrees
- moved D201 2.22 mm to (137.6, 73.3)
- moved C208 1.01 mm to (156.2, 76.4)
- moved U201 1.01 mm to (150.7, 77.3)
- renumbered C201 to C200, C211 to C201, C206 to C203, C209 to C204, C213 to C205, C210 to C206, C204 to C208, C212 to C209, C214 to C211, C217 to C212, C218 to C213, C216 to C214, C221 to C215, C219 to C216, C220 to C217, C215 to C218, C224 to C219, C222 to C220, C223 to C221, C232 to C222, C225 to C223, C226 to C224, C229 to C225, C228 to C226, C230 to C227, C231 to C228, C227 to C229, C233 to C230, D200 to D201, D201 to D202, J201 to J200, J200 to J201, J203 to J202, J202 to J203, J207 to J205, J205 to J206, J206 to J207, R201 to R200, R202 to R201, R203 to R202, R204 to R203, R200 to R204, R217 to R214, R214 to R215, R215 to R217, U205 to U204, U204 to U205
Routing:
- net STM32_BOOT: track 39.4 -> 41.5 mm
- net GND: track 81.1 -> 79.5 mm, vias 37 -> 35
- net +5V: track 25.6 -> 24.3 mm
- net STM32_USART1_RX: track 45.4 -> 44.1 mm, vias 2 -> 1
- net STM32_USART1_TX: track 43.7 -> 44.0 mm, vias 2 -> 1

Commit message: feat: change crystal
Parts:
- removed X200: XVFEELNANF-8MHZ, easyeda2kicad:CRYSTAL-SMD_4P-L5.0-W3.2-BL-1
- added X201: X32258MOB4SI, easyeda2kicad:CRYSTAL-SMD_4P-L3.2-W2.5-BL, F.Cu at (135.6, 90.7)
- C200, C218: value 22pF -> 18pF
- R206: value 10K -> 1K
- moved C218 1.79 mm to (135.3, 93.5), turned to 0 degrees
- moved C200 0.52 mm to (135.9, 88.0), turned to 180 degrees
- moved G*** 0.36 mm to (135.3, 97.4)
Connections:
- R212 pad 1: +3.3V -> STM32_NRST
Routing:
- net STM32_NRST: track 27.0 -> 39.4 mm, vias 2 -> 3
- net STM32_XTAL_IN: track 18.6 -> 14.9 mm
- net GND: track 79.5 -> 81.9 mm, vias 35 -> 36
- net STM32_XTAL_OUT: track 10.3 -> 12.3 mm
- net +3.3V: track 85.4 -> 84.4 mm, vias 24 -> 23
